File: REF1256.kicad_sch (KiCad schematic)
At the start: 13 parts, among them J1 Gameboy Cartridge Connector, J2 N64 Cartridge Slot, J3 Edge_Connector, SW1 SW_Push, U1 LZ9FC17, U2 SN74HC32N, U3 SST28LF040, U4 SST28LF040, U5 LM78L05_SO8

Commit message: Add files via upload
Parts:
- C1, C2: value C_Small -> 100 nF
Other:
- note removed: ""A15" on the game boy cartridge connector isn't exactly A15 from the CPU. It's a signal that's low when the Game Boy is accessing $0000-$7FFF, but its timing is different from the rest of the address bus and it acts more like a bus enable signal. Similarly, "CS" is low when the Game Boy is accessing $A000-$FDFF, but it shares this same different timing with "A15"."
Changed lines of the file:
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@@
 		)
 	)
-	(text "\"A15\" on the game boy cartridge connector isn't exactly A15 from the CPU.\nIt's a signal that's low when the Game Boy is accessing $0000-$7FFF,\nbut its timing is different from the rest of the address bus and it acts \nmore like a bus enable signal. Similarly, \"CS\" is low when the Game Boy \nis accessing $A000-$FDFF, but it shares this same different timing with \"A15\".\n"
-		(exclude_from_sim no)
-		(at 132.842 170.942 0)
-		(effects
-			(font
-				(size 1.27 1.27)
-			)
-		)
-	)
 	(label "A14"
 		(at 64.77 113.03 0)
@@
 			)
 		)
-		(property "Value" "C_Small"
+		(property "Value" "100 nF"
 			(at 368.3 116.8462 0)
 			(effects
@@
 			)
 		)
-		(property "Value" "C_Small"
+		(property "Value" "100 nF"
 			(at 362.458 165.354 0)
 			(effects
